Commit message: URDF tree naming changed, the cabinets are hollow

File: ros2_ws/src/manipulator_description/urdf/box_placement_frames.urdf.xacro (robot description, xacro)
@@ -85,10 +85,13 @@
       <xacro:property name="frame_y" value="0.0"/>
       <!-- Create frame link (no geometry, just coordinate frame) -->
-      <link name="${side}_cab${cabinet_num}_box_placement_${current_row}_${current_col}"/>
+      <!-- Simplified naming: addr_{side_abbrev}_{cab}_{row}_{col} -->
+      <!-- Example: addr_l_1_2_3 = left row, cabinet 1, row 2, column 3 -->
+      <xacro:property name="side_abbrev" value="${'l' if side == 'left' else 'r'}"/>
+      <link name="addr_${side_abbrev}_${cabinet_num}_${current_row}_${current_col}"/>
       <!-- Attach to cabinet -->
-      <joint name="${side}_cab${cabinet_num}_box_placement_${current_row}_${current_col}_to_cabinet"
+      <joint name="addr_${side_abbrev}_${cabinet_num}_${current_row}_${current_col}_to_cab"
              type="fixed">
         <parent link="${parent_link}"/>
-        <child link="${side}_cab${cabinet_num}_box_placement_${current_row}_${current_col}"/>
+        <child link="addr_${side_abbrev}_${cabinet_num}_${current_row}_${current_col}"/>
         <origin xyz="${frame_x} ${frame_y} ${frame_z}" rpy="0 0 0"/>
       </joint>

File: ros2_ws/src/manipulator_description/urdf/cabinet.urdf.xacro (robot description, xacro)
@@ -32,4 +32,7 @@
     <xacro:property name="cab_y" value="${cab_dims['exterior']['y']}"/>
     <xacro:property name="cab_z" value="${cab_dims['exterior']['z']}"/>
+    <!-- Simplified cabinet naming: cab_{side_abbrev}_{num} -->
+    <!-- Example: cab_l_1 = left row, cabinet 1 -->
+    <xacro:property name="side_abbrev" value="${'l' if side == 'left' else 'r'}"/>
     <!-- Cabinet link -->
     <!-- Origin is at left-bottom-front corner (for left row) or right-bottom-front corner (for right row) -->
@@ -41,20 +44,74 @@
     <xacro:property name="visual_offset_y" value="${cab_y / 2.0}"/>
     <xacro:property name="visual_offset_z" value="${cab_z / 2.0}"/>
-    <link name="${side}_cab${cabinet_num}">
-      <visual>
-        <!-- Offset box center to align with corner origin -->
-        <origin xyz="${visual_offset_x} ${visual_offset_y} ${visual_offset_z}" rpy="0 0 0"/>
-        <geometry>
-          <xacro:if value="${cabinet_model is not None and cabinet_model.get('mesh', None) is not None}">
+    <!-- Cabinet dimensions for hollow construction -->
+    <xacro:property name="wall_thick" value="${cab_dims['wall_thickness']}"/>
+    <xacro:property name="interior_x" value="${cab_dims['interior']['x']}"/>
+    <xacro:property name="interior_y" value="${cab_dims['interior']['y']}"/>
+    <xacro:property name="interior_z" value="${cab_dims['interior']['z']}"/>
+    <link name="cab_${side_abbrev}_${cabinet_num}">
+      <!-- Use mesh if available, otherwise create hollow box from primitives -->
+      <xacro:if value="${cabinet_model is not None and cabinet_model.get('mesh', None) is not None}">
+        <visual>
+          <origin xyz="${visual_offset_x} ${visual_offset_y} ${visual_offset_z}" rpy="0 0 0"/>
+          <geometry>
             <mesh filename="${cabinet_model['mesh']['visual']}" scale="1 1 1"/>
-          </xacro:if>
-          <xacro:unless value="${cabinet_model is not None and cabinet_model.get('mesh', None) is not None}">
-            <box size="${cab_x} ${cab_y} ${cab_z}"/>
-          </xacro:unless>
-        </geometry>
-        <material name="cabinet_grey"/>
-      </visual>
+          </geometry>
+          <material name="cabinet_grey"/>
+        </visual>
+      </xacro:if>
+      <xacro:unless value="${cabinet_model is not None and cabinet_model.get('mesh', None) is not None}">
+        <!-- Hollow cabinet made from 6 walls (bottom, top, left, right, back, front-frame) -->
+        <!-- Bottom wall -->
+        <visual name="bottom">
+          <origin xyz="${cab_x/2.0} ${cab_y/2.0} ${wall_thick/2.0}" rpy="0 0 0"/>
+          <geometry>
+            <box size="${cab_x} ${cab_y} ${wall_thick}"/>
+          </geometry>
+          <material name="cabinet_grey"/>
+        </visual>
+        <!-- Top wall -->
+        <visual name="top">
+          <origin xyz="${cab_x/2.0} ${cab_y/2.0} ${cab_z - wall_thick/2.0}" rpy="0 0 0"/>
+          <geometry>
+            <box size="${cab_x} ${cab_y} ${wall_thick}"/>
+          </geometry>
+          <material name="cabinet_grey"/>
+        </visual>
+        <!-- Left wall -->
+        <visual name="left">
+          <origin xyz="${wall_thick/2.0} ${cab_y/2.0} ${cab_z/2.0}" rpy="0 0 0"/>
+          <geometry>
+            <box size="${wall_thick} ${cab_y} ${cab_z}"/>
+          </geometry>
+          <material name="cabinet_grey"/>
+        </visual>
+        <!-- Right wall -->
+        <visual name="right">
+          <origin xyz="${cab_x - wall_thick/2.0} ${cab_y/2.0} ${cab_z/2.0}" rpy="0 0 0"/>
+          <geometry>
+            <box size="${wall_thick} ${cab_y} ${cab_z}"/>
+          </geometry>
+          <material name="cabinet_grey"/>
+        </visual>
+        <!-- Back wall -->
+        <visual name="back">
+          <origin xyz="${cab_x/2.0} ${cab_y - wall_thick/2.0} ${cab_z/2.0}" rpy="0 0 0"/>
+          <geometry>
+            <box size="${cab_x} ${wall_thick} ${cab_z}"/>
+          </geometry>
+          <material name="cabinet_grey"/>
+        </visual>
+        <!-- Front opening (just frame, no solid wall - boxes slide through here) -->
+        <!-- Top frame bar -->
+        <visual name="front_top">
+          <origin xyz="${cab_x/2.0} ${wall_thick/2.0} ${cab_z - wall_thick/2.0}" rpy="0 0 0"/>
+          <geometry>
+            <box size="${cab_x} ${wall_thick} ${wall_thick}"/>
+          </geometry>
+          <material name="cabinet_grey"/>
+        </visual>
+      </xacro:unless>
+      <!-- Collision: simplified box (for now, can be refined later) -->
       <collision>
-        <!-- Same offset for collision -->
         <origin xyz="${visual_offset_x} ${visual_offset_y} ${visual_offset_z}" rpy="0 0 0"/>
         <geometry>
@@ -74,7 +131,7 @@
     </link>
     <!-- Fixed joint to parent row -->
-    <joint name="${side}_cab${cabinet_num}_to_row" type="fixed">
+    <joint name="cab_${side_abbrev}_${cabinet_num}_to_row" type="fixed">
       <parent link="${parent_link}"/>
-      <child link="${side}_cab${cabinet_num}"/>
+      <child link="cab_${side_abbrev}_${cabinet_num}"/>
       <origin xyz="${position_x} ${position_y} ${position_z}" rpy="0 0 ${rotation_z}"/>
     </joint>
@@ -87,5 +144,5 @@
       num_depts="${num_depts}"
       config="${config}"
-      parent_link="${side}_cab${cabinet_num}"/>
+      parent_link="cab_${side_abbrev}_${cabinet_num}"/>
   </xacro:macro>
 </robot>

File: ros2_ws/src/manipulator_description/urdf/cabinet_row.urdf.xacro (robot description, xacro)
@@ -11,10 +11,12 @@
     <xacro:property name="row_offset" value="${row_config['offset']}"/>
     <xacro:property name="cabinets" value="${row_config['cabinets']}"/>
+    <!-- Simplified side naming: side_l or side_r -->
+    <xacro:property name="side_abbrev" value="${'l' if side == 'left' else 'r'}"/>
     <!-- Row base link -->
-    <link name="${side}_cabinet_row_base"/>
+    <link name="side_${side_abbrev}"/>
     <!-- Fixed joint to parent -->
-    <joint name="${side}_cabinet_row_to_parent" type="fixed">
+    <joint name="side_${side_abbrev}_to_base" type="fixed">
       <parent link="${parent_link}"/>
-      <child link="${side}_cabinet_row_base"/>
+      <child link="side_${side_abbrev}"/>
       <origin xyz="${row_offset['x']} ${row_offset['y']} ${row_offset['z']}" rpy="0 0 0"/>
     </joint>
@@ -38,5 +40,5 @@
         cabinet_num="1"
         size_name="${cab1_size}"
-        parent_link="${side}_cabinet_row_base"
+        parent_link="side_${side_abbrev}"
         position_x="${cab1_x}"
         position_y="${cab1_y}"

Commit message: The boxes for the addresses are created

File: ros2_ws/src/manipulator_description/urdf/box_placement_frames.urdf.xacro (robot description, xacro)
@@ -18,4 +18,10 @@
     <xacro:property name="box_col_config" value="${config['box_configurations']['columns_' + str(num_cols)]}"/>
     <xacro:property name="box_row_config" value="${config['box_configurations']['rows_' + str(num_rows)]}"/>
+    <!-- Get visualization settings -->
+    <xacro:property name="viz_config" value="${config['visualization']}"/>
+    <xacro:property name="show_boxes" value="${viz_config['show_address_boxes']}"/>
+    <xacro:property name="box_width" value="${box_col_config['width']}"/>
+    <xacro:property name="box_depth" value="${config['department_configurations']['departments_' + str(num_depts)]['depth'] * num_depts}"/>
+    <xacro:property name="box_height" value="${box_row_config['height']}"/>
     <!-- Generate placement frames using recursive macros -->
     <xacro:placement_rows
@@ -27,5 +33,9 @@
       parent_link="${parent_link}"
       box_col_config="${box_col_config}"
-      box_row_config="${box_row_config}"/>
+      box_row_config="${box_row_config}"
+      show_boxes="${show_boxes}"
+      box_width="${box_width}"
+      box_depth="${box_depth}"
+      box_height="${box_height}"/>
   </xacro:macro>
   <!-- Recursion for rows -->
@@ -38,5 +48,9 @@
     parent_link
     box_col_config
-    box_row_config">
+    box_row_config
+    show_boxes
+    box_width
+    box_depth
+    box_height">
     <xacro:if value="${current_row &lt;= max_rows}">
       <!-- Create frames for all columns in this row -->
@@ -50,5 +64,9 @@
         parent_link="${parent_link}"
         box_col_config="${box_col_config}"
-        box_row_config="${box_row_config}"/>
+        box_row_config="${box_row_config}"
+        show_boxes="${show_boxes}"
+        box_width="${box_width}"
+        box_depth="${box_depth}"
+        box_height="${box_height}"/>
       <!-- Recurse for next row -->
       <xacro:placement_rows
@@ -60,5 +78,9 @@
         parent_link="${parent_link}"
         box_col_config="${box_col_config}"
-        box_row_config="${box_row_config}"/>
+        box_row_config="${box_row_config}"
+        show_boxes="${show_boxes}"
+        box_width="${box_width}"
+        box_depth="${box_depth}"
+        box_height="${box_height}"/>
     </xacro:if>
   </xacro:macro>
@@ -73,5 +95,9 @@
     parent_link
     box_col_config
-    box_row_config">
+    box_row_config
+    show_boxes
+    box_width
+    box_depth
+    box_height">
     <xacro:if value="${current_col &lt;= max_cols}">
       <!-- Calculate frame position (v2.2 formulas) -->
@@ -84,9 +110,21 @@
       <!-- Y: At front of cabinet (0.0 in cabinet local frame) -->
       <xacro:property name="frame_y" value="0.0"/>
-      <!-- Create frame link (no geometry, just coordinate frame) -->
+      <!-- Create frame link -->
       <!-- Simplified naming: addr_{side_abbrev}_{cab}_{row}_{col} -->
       <!-- Example: addr_l_1_2_3 = left row, cabinet 1, row 2, column 3 -->
       <xacro:property name="side_abbrev" value="${'l' if side == 'left' else 'r'}"/>
-      <link name="addr_${side_abbrev}_${cabinet_num}_${current_row}_${current_col}"/>
+      <link name="addr_${side_abbrev}_${cabinet_num}_${current_row}_${current_col}">
+        <!-- Optional: Show box visual for testing -->
+        <!-- Box centered at address frame origin -->
+        <xacro:if value="${show_boxes}">
+          <visual>
+            <origin xyz="0 ${box_depth/2.0} 0" rpy="0 0 0"/>
+            <geometry>
+              <box size="${box_width} ${box_depth} ${box_height}"/>
+            </geometry>
+            <material name="box_light_blue"/>
+          </visual>
+        </xacro:if>
+      </link>
       <!-- Attach to cabinet -->
       <joint name="addr_${side_abbrev}_${cabinet_num}_${current_row}_${current_col}_to_cab"
@@ -106,5 +144,9 @@
         parent_link="${parent_link}"
         box_col_config="${box_col_config}"
-        box_row_config="${box_row_config}"/>
+        box_row_config="${box_row_config}"
+        show_boxes="${show_boxes}"
+        box_width="${box_width}"
+        box_depth="${box_depth}"
+        box_height="${box_height}"/>
     </xacro:if>
   </xacro:macro>

File: ros2_ws/src/manipulator_description/urdf/materials.xacro (robot description, xacro)
@@ -7,4 +7,13 @@
   <material name="box_blue">
     <color rgba="0.3 0.5 0.8 1.0"/>
+  </material>
+  <material name="box_light_blue">
+    <color rgba="0.53 0.81 0.92 1.0"/>  <!-- Light sky blue -->
+  </material>
+  <material name="box_green">
+    <color rgba="0.0 1.0 0.0 0.7"/>  <!-- Green, semi-transparent for target -->
+  </material>
+  <material name="box_scarlet">
+    <color rgba="1.0 0.14 0.0 0.7"/>  <!-- Scarlet red, semi-transparent for empty -->
   </material>
   <material name="department_marker_red">
