Commit message: Basic manipulator urdf added and works

File: ros2_ws/src/manipulator_description/urdf/robot.urdf.xacro (robot description, xacro)
@@ -4,6 +4,6 @@
     Top-level URDF for the complete robotic manipulator system
     This file assembles:
+    - Manipulator (base + selector + picker assemblies)
     - Storage system (cabinets + placement frames)
-    - Manipulator (TODO: to be added later)
     Usage:
       xacro robot.urdf.xacro > robot.urdf
@@ -12,26 +12,13 @@
   <!-- Load materials -->
   <xacro:include filename="$(find manipulator_description)/urdf/materials.xacro"/>
+  <!-- Load manipulator -->
+  <xacro:include filename="$(find manipulator_description)/urdf/manipulator/manipulator.urdf.xacro"/>
   <!-- Load storage system -->
   <xacro:include filename="$(find manipulator_description)/urdf/storage_system.urdf.xacro"/>
   <!-- World link (reference frame) -->
   <link name="world"/>
-  <!-- Base link (manipulator base, origin of our coordinate system) -->
-  <link name="base_link">
-    <visual>
-      <geometry>
-        <cylinder radius="0.1" length="0.05"/>
-      </geometry>
-      <material name="manipulator_dark_grey"/>
-    </visual>
-    <collision>
-      <geometry>
-        <cylinder radius="0.1" length="0.05"/>
-      </geometry>
-    </collision>
-    <inertial>
-      <mass value="10.0"/>
-      <inertia ixx="1.0" ixy="0.0" ixz="0.0" iyy="1.0" iyz="0.0" izz="1.0"/>
-    </inertial>
-  </link>
+  <!-- Instantiate manipulator (creates base_link and entire manipulator tree) -->
+  <xacro:manipulator
+    config_file="$(find manipulator_description)/config/manipulator_params.yaml"/>
   <!-- Fixed joint: world -> base_link -->
   <joint name="world_to_base" type="fixed">
@@ -40,10 +27,7 @@
     <origin xyz="0 0 0" rpy="0 0 0"/>
   </joint>
-  <!-- Storage system -->
+  <!-- Storage system (attached to world) -->
   <xacro:storage_system
-    parent_link="base_link"
+    parent_link="world"
     config_file="$(find manipulator_description)/config/storage_params.yaml"/>
-  <!-- TODO: Manipulator will be added here later -->
-  <!-- <xacro:include filename="$(find manipulator_description)/urdf/manipulator.urdf.xacro"/> -->
-  <!-- <xacro:manipulator parent_link="base_link"/> -->
 </robot>

Commit message: Epic 7 HW interface is ready for implementation

File: ros2_ws/src/manipulator_description/urdf/robot.urdf.xacro (robot description, xacro)
@@ -26,5 +26,5 @@
     <parent link="world"/>
     <child link="base_link"/>
-    <origin xyz="0 0 0.09" rpy="0 0 0"/>
+    <origin xyz="-1.0 0 0.09" rpy="0 0 0"/>
   </joint>
   <!-- Storage system (attached to world) -->
