Commit message: meshes paths via yaml added

File: ros2_ws/src/manipulator_description/urdf/manipulator/manipulator_base.urdf.xacro (robot description, xacro)
@@ -21,5 +21,5 @@
         <origin xyz="0 0 0" rpy="0 0 0"/>
         <geometry>
-          <mesh filename="file://$(find manipulator_description)/meshes/manipulator/base_link.STL"/>
+          <mesh filename="file://$(find manipulator_description)/meshes/manipulator/${base['base_link']['mesh']}"/>
         </geometry>
         <material name="base_link_color">
@@ -31,5 +31,5 @@
         <origin xyz="0 0 0" rpy="0 0 0"/>
         <geometry>
-          <mesh filename="file://$(find manipulator_description)/meshes/manipulator/base_link.STL"/>
+          <mesh filename="file://$(find manipulator_description)/meshes/manipulator/${base['base_link']['mesh']}"/>
         </geometry>
       </collision>
@@ -61,5 +61,5 @@
         <origin xyz="0 0 0" rpy="0 0 0"/>
         <geometry>
-          <mesh filename="file://$(find manipulator_description)/meshes/manipulator/main_frame.STL"/>
+          <mesh filename="file://$(find manipulator_description)/meshes/manipulator/${base['main_frame']['mesh']}"/>
         </geometry>
         <material name="main_frame_color">
@@ -71,5 +71,5 @@
         <origin xyz="0 0 0" rpy="0 0 0"/>
         <geometry>
-          <mesh filename="file://$(find manipulator_description)/meshes/manipulator/main_frame.STL"/>
+          <mesh filename="file://$(find manipulator_description)/meshes/manipulator/${base['main_frame']['mesh']}"/>
         </geometry>
       </collision>

File: ros2_ws/src/manipulator_description/urdf/manipulator/manipulator_picker.urdf.xacro (robot description, xacro)
@@ -22,5 +22,5 @@
         <origin xyz="0 0 0" rpy="0 0 0"/>
         <geometry>
-          <mesh filename="file://$(find manipulator_description)/meshes/manipulator/picker_frame.STL"/>
+          <mesh filename="file://$(find manipulator_description)/meshes/manipulator/${picker['picker_frame']['mesh']}"/>
         </geometry>
         <material name="picker_frame_color">
@@ -32,5 +32,5 @@
         <origin xyz="0 0 0" rpy="0 0 0"/>
         <geometry>
-          <mesh filename="file://$(find manipulator_description)/meshes/manipulator/picker_frame.STL"/>
+          <mesh filename="file://$(find manipulator_description)/meshes/manipulator/${picker['picker_frame']['mesh']}"/>
         </geometry>
       </collision>
@@ -87,5 +87,5 @@
         <origin xyz="0 0 0" rpy="0 0 0"/>
         <geometry>
-          <mesh filename="file://$(find manipulator_description)/meshes/manipulator/picker_rail.STL"/>
+          <mesh filename="file://$(find manipulator_description)/meshes/manipulator/${picker['picker_rail']['mesh']}"/>
         </geometry>
         <material name="picker_rail_color">
@@ -97,5 +97,5 @@
         <origin xyz="0 0 0" rpy="0 0 0"/>
         <geometry>
-          <mesh filename="file://$(find manipulator_description)/meshes/manipulator/picker_rail.STL"/>
+          <mesh filename="file://$(find manipulator_description)/meshes/manipulator/${picker['picker_rail']['mesh']}"/>
         </geometry>
       </collision>
@@ -152,5 +152,5 @@
         <origin xyz="0 0 0" rpy="0 0 0"/>
         <geometry>
-          <mesh filename="file://$(find manipulator_description)/meshes/manipulator/picker_base.STL"/>
+          <mesh filename="file://$(find manipulator_description)/meshes/manipulator/${picker['picker_base']['mesh']}"/>
         </geometry>
         <material name="picker_base_color">
@@ -162,5 +162,5 @@
         <origin xyz="0 0 0" rpy="0 0 0"/>
         <geometry>
-          <mesh filename="file://$(find manipulator_description)/meshes/manipulator/picker_base.STL"/>
+          <mesh filename="file://$(find manipulator_description)/meshes/manipulator/${picker['picker_base']['mesh']}"/>
         </geometry>
       </collision>
@@ -217,5 +217,5 @@
         <origin xyz="0 0 0" rpy="0 0 0"/>
         <geometry>
-          <mesh filename="file://$(find manipulator_description)/meshes/manipulator/picker_jaw.STL"/>
+          <mesh filename="file://$(find manipulator_description)/meshes/manipulator/${picker['picker_jaw']['mesh']}"/>
         </geometry>
         <material name="picker_jaw_color">
@@ -227,5 +227,5 @@
         <origin xyz="0 0 0" rpy="0 0 0"/>
         <geometry>
-          <mesh filename="file://$(find manipulator_description)/meshes/manipulator/picker_jaw.STL"/>
+          <mesh filename="file://$(find manipulator_description)/meshes/manipulator/${picker['picker_jaw']['mesh']}"/>
         </geometry>
       </collision>

File: ros2_ws/src/manipulator_description/urdf/manipulator/manipulator_selector.urdf.xacro (robot description, xacro)
@@ -23,5 +23,5 @@
         <origin xyz="0 0 0" rpy="0 0 0"/>
         <geometry>
-          <mesh filename="file://$(find manipulator_description)/meshes/manipulator/selector_frame.STL"/>
+          <mesh filename="file://$(find manipulator_description)/meshes/manipulator/${selector['selector_frame']['mesh']}"/>
         </geometry>
         <material name="selector_frame_color">
@@ -33,5 +33,5 @@
         <origin xyz="0 0 0" rpy="0 0 0"/>
         <geometry>
-          <mesh filename="file://$(find manipulator_description)/meshes/manipulator/selector_frame.STL"/>
+          <mesh filename="file://$(find manipulator_description)/meshes/manipulator/${selector['selector_frame']['mesh']}"/>
         </geometry>
       </collision>
@@ -92,5 +92,5 @@
         <origin xyz="0 0 0" rpy="0 0 0"/>
         <geometry>
-          <mesh filename="file://$(find manipulator_description)/meshes/manipulator/left_container_jaw.STL"/>
+          <mesh filename="file://$(find manipulator_description)/meshes/manipulator/${selector['left_container_jaw']['mesh']}"/>
         </geometry>
         <material name="left_container_jaw_color">
@@ -102,5 +102,5 @@
         <origin xyz="0 0 0" rpy="0 0 0"/>
         <geometry>
-          <mesh filename="file://$(find manipulator_description)/meshes/manipulator/left_container_jaw.STL"/>
+          <mesh filename="file://$(find manipulator_description)/meshes/manipulator/${selector['left_container_jaw']['mesh']}"/>
         </geometry>
       </collision>
@@ -157,5 +157,5 @@
         <origin xyz="0 0 0" rpy="0 0 0"/>
         <geometry>
-          <mesh filename="file://$(find manipulator_description)/meshes/manipulator/right_container_jaw.STL"/>
+          <mesh filename="file://$(find manipulator_description)/meshes/manipulator/${selector['right_container_jaw']['mesh']}"/>
         </geometry>
         <material name="right_container_jaw_color">
@@ -167,5 +167,5 @@
         <origin xyz="0 0 0" rpy="0 0 0"/>
         <geometry>
-          <mesh filename="file://$(find manipulator_description)/meshes/manipulator/right_container_jaw.STL"/>
+          <mesh filename="file://$(find manipulator_description)/meshes/manipulator/${selector['right_container_jaw']['mesh']}"/>
         </geometry>
       </collision>
@@ -227,5 +227,5 @@
         <origin xyz="0 0 0" rpy="0 0 0"/>
         <geometry>
-          <mesh filename="file://$(find manipulator_description)/meshes/manipulator/gripper.STL"/>
+          <mesh filename="file://$(find manipulator_description)/meshes/manipulator/${selector['gripper']['mesh']}"/>
         </geometry>
         <material name="gripper_color">
@@ -237,5 +237,5 @@
         <origin xyz="0 0 0" rpy="0 0 0"/>
         <geometry>
-          <mesh filename="file://$(find manipulator_description)/meshes/manipulator/gripper.STL"/>
+          <mesh filename="file://$(find manipulator_description)/meshes/manipulator/${selector['gripper']['mesh']}"/>
         </geometry>
       </collision>

File: ros2_ws/src/manipulator_description/urdf/robot.urdf.xacro (robot description, xacro)
@@ -26,5 +26,5 @@
     <parent link="world"/>
     <child link="base_link"/>
-    <origin xyz="0 0 0" rpy="0 0 0"/>
+    <origin xyz="0 0 0.09" rpy="0 0 0"/>
   </joint>
   <!-- Storage system (attached to world) -->
