Commit message: joystick control implemented 80%. gravity issue solved in gazebo - used to lock vertical joints

File: ros2_ws/src/manipulator_description/urdf/manipulator/manipulator_selector.urdf.xacro (robot description, xacro)
@@ -213,9 +213,5 @@
         damping="${selector['selector_right_container_jaw_joint']['dynamics']['damping']}"
         friction="${selector['selector_right_container_jaw_joint']['dynamics']['friction']}"/>
-      <!-- MIMIC: Right jaw mirrors left jaw movement -->
-      <mimic
-        joint="${selector['selector_right_container_jaw_joint']['mimic']['joint']}"
-        multiplier="${selector['selector_right_container_jaw_joint']['mimic']['multiplier']}"
-        offset="${selector['selector_right_container_jaw_joint']['mimic']['offset']}"/>
+      <!-- MIMIC REMOVED: dartsim doesn't support mimic joints, controlled independently via joy_control -->
     </joint>
     <!-- ================================================================ -->

File: ros2_ws/src/manipulator_description/urdf/manipulator/ros2_control.xacro (robot description, xacro)
@@ -14,4 +14,7 @@
         <hardware>
           <plugin>gz_ros2_control/GazeboSimSystem</plugin>
+          <!-- PID gains for position control (especially important for vertical joints fighting gravity) -->
+          <param name="hold_joints">true</param>
+          <param name="position_proportional_gain">50.0</param>
         </hardware>
       </xacro:if>
@@ -47,5 +50,5 @@
       <joint name="main_frame_selector_frame_joint">
         <command_interface name="position">
-          <param name="min">0.0</param>
+          <param name="min">-0.01</param>
           <param name="max">1.5</param>
         </command_interface>
@@ -55,9 +58,9 @@
         </command_interface>
         <state_interface name="position">
-          <param name="initial_value">0.0</param>
+          <param name="initial_value">0.05</param>
         </state_interface>
         <state_interface name="velocity"/>
       </joint>
-      <!-- selector_left_container_jaw_joint (Y-axis gripper) -->
+      <!-- selector_left_container_jaw_joint (left container jaw) -->
       <joint name="selector_left_container_jaw_joint">
         <command_interface name="position">
@@ -74,5 +77,20 @@
         <state_interface name="velocity"/>
       </joint>
-      <!-- Note: selector_right_container_jaw_joint is mimic, not controlled directly -->
+      <!-- selector_right_container_jaw_joint (right container jaw) -->
+      <!-- Note: Was mimic joint, but dartsim doesn't support mimic, so controlled independently -->
+      <joint name="selector_right_container_jaw_joint">
+        <command_interface name="position">
+          <param name="min">-0.2</param>
+          <param name="max">0.2</param>
+        </command_interface>
+        <command_interface name="velocity">
+          <param name="min">-1.0</param>
+          <param name="max">1.0</param>
+        </command_interface>
+        <state_interface name="position">
+          <param name="initial_value">0.0</param>
+        </state_interface>
+        <state_interface name="velocity"/>
+      </joint>
       <!-- selector_frame_gripper_joint (Y-axis magnet holder) -->
       <joint name="selector_frame_gripper_joint">
@@ -96,5 +114,5 @@
       <joint name="selector_frame_picker_frame_joint">
         <command_interface name="position">
-          <param name="min">0.0</param>
+          <param name="min">-0.01</param>
           <param name="max">0.3</param>
         </command_interface>
@@ -104,5 +122,5 @@
         </command_interface>
         <state_interface name="position">
-          <param name="initial_value">0.0</param>
+          <param name="initial_value">0.05</param>
         </state_interface>
         <state_interface name="velocity"/>
