Commit message: Gazebosimulation added

File: ros2_ws/src/manipulator_description/urdf/manipulator/manipulator.urdf.xacro (robot description, xacro)
@@ -16,6 +16,7 @@
   <xacro:include filename="$(find manipulator_description)/urdf/manipulator/manipulator_selector.urdf.xacro"/>
   <xacro:include filename="$(find manipulator_description)/urdf/manipulator/manipulator_picker.urdf.xacro"/>
+  <xacro:include filename="$(find manipulator_description)/urdf/manipulator/ros2_control.xacro"/>
   <!-- Main manipulator macro -->
-  <xacro:macro name="manipulator" params="config_file">
+  <xacro:macro name="manipulator" params="config_file sim:=true">
     <!--
       Assembly hierarchy:
@@ -45,4 +46,8 @@
       parent_link="selector_frame"
       config_file="${config_file}"/>
+    <!-- 4. ROS2 CONTROL: Hardware interfaces and controllers -->
+    <xacro:manipulator_ros2_control
+      name="manipulator_system"
+      sim="${sim}"/>
   </xacro:macro>
 </robot>

File: ros2_ws/src/manipulator_description/urdf/manipulator/manipulator_base.urdf.xacro (robot description, xacro)
@@ -21,5 +21,5 @@
         <origin xyz="0 0 0" rpy="0 0 0"/>
         <geometry>
-          <mesh filename="${base['base_link']['mesh']}"/>
+          <mesh filename="file://$(find manipulator_description)/meshes/manipulator/base_link.STL"/>
         </geometry>
         <material name="base_link_color">
@@ -31,5 +31,5 @@
         <origin xyz="0 0 0" rpy="0 0 0"/>
         <geometry>
-          <mesh filename="${base['base_link']['mesh']}"/>
+          <mesh filename="file://$(find manipulator_description)/meshes/manipulator/base_link.STL"/>
         </geometry>
       </collision>
@@ -61,5 +61,5 @@
         <origin xyz="0 0 0" rpy="0 0 0"/>
         <geometry>
-          <mesh filename="${base['main_frame']['mesh']}"/>
+          <mesh filename="file://$(find manipulator_description)/meshes/manipulator/main_frame.STL"/>
         </geometry>
         <material name="main_frame_color">
@@ -71,5 +71,5 @@
         <origin xyz="0 0 0" rpy="0 0 0"/>
         <geometry>
-          <mesh filename="${base['main_frame']['mesh']}"/>
+          <mesh filename="file://$(find manipulator_description)/meshes/manipulator/main_frame.STL"/>
         </geometry>
       </collision>

File: ros2_ws/src/manipulator_description/urdf/manipulator/manipulator_picker.urdf.xacro (robot description, xacro)
@@ -22,5 +22,5 @@
         <origin xyz="0 0 0" rpy="0 0 0"/>
         <geometry>
-          <mesh filename="${picker['picker_frame']['mesh']}"/>
+          <mesh filename="file://$(find manipulator_description)/meshes/manipulator/picker_frame.STL"/>
         </geometry>
         <material name="picker_frame_color">
@@ -32,5 +32,5 @@
         <origin xyz="0 0 0" rpy="0 0 0"/>
         <geometry>
-          <mesh filename="${picker['picker_frame']['mesh']}"/>
+          <mesh filename="file://$(find manipulator_description)/meshes/manipulator/picker_frame.STL"/>
         </geometry>
       </collision>
@@ -87,5 +87,5 @@
         <origin xyz="0 0 0" rpy="0 0 0"/>
         <geometry>
-          <mesh filename="${picker['picker_rail']['mesh']}"/>
+          <mesh filename="file://$(find manipulator_description)/meshes/manipulator/picker_rail.STL"/>
         </geometry>
         <material name="picker_rail_color">
@@ -97,5 +97,5 @@
         <origin xyz="0 0 0" rpy="0 0 0"/>
         <geometry>
-          <mesh filename="${picker['picker_rail']['mesh']}"/>
+          <mesh filename="file://$(find manipulator_description)/meshes/manipulator/picker_rail.STL"/>
         </geometry>
       </collision>
@@ -152,5 +152,5 @@
         <origin xyz="0 0 0" rpy="0 0 0"/>
         <geometry>
-          <mesh filename="${picker['picker_base']['mesh']}"/>
+          <mesh filename="file://$(find manipulator_description)/meshes/manipulator/picker_base.STL"/>
         </geometry>
         <material name="picker_base_color">
@@ -162,5 +162,5 @@
         <origin xyz="0 0 0" rpy="0 0 0"/>
         <geometry>
-          <mesh filename="${picker['picker_base']['mesh']}"/>
+          <mesh filename="file://$(find manipulator_description)/meshes/manipulator/picker_base.STL"/>
         </geometry>
       </collision>
@@ -217,5 +217,5 @@
         <origin xyz="0 0 0" rpy="0 0 0"/>
         <geometry>
-          <mesh filename="${picker['picker_jaw']['mesh']}"/>
+          <mesh filename="file://$(find manipulator_description)/meshes/manipulator/picker_jaw.STL"/>
         </geometry>
         <material name="picker_jaw_color">
@@ -227,5 +227,5 @@
         <origin xyz="0 0 0" rpy="0 0 0"/>
         <geometry>
-          <mesh filename="${picker['picker_jaw']['mesh']}"/>
+          <mesh filename="file://$(find manipulator_description)/meshes/manipulator/picker_jaw.STL"/>
         </geometry>
       </collision>

File: ros2_ws/src/manipulator_description/urdf/manipulator/manipulator_selector.urdf.xacro (robot description, xacro)
@@ -23,5 +23,5 @@
         <origin xyz="0 0 0" rpy="0 0 0"/>
         <geometry>
-          <mesh filename="${selector['selector_frame']['mesh']}"/>
+          <mesh filename="file://$(find manipulator_description)/meshes/manipulator/selector_frame.STL"/>
         </geometry>
         <material name="selector_frame_color">
@@ -33,5 +33,5 @@
         <origin xyz="0 0 0" rpy="0 0 0"/>
         <geometry>
-          <mesh filename="${selector['selector_frame']['mesh']}"/>
+          <mesh filename="file://$(find manipulator_description)/meshes/manipulator/selector_frame.STL"/>
         </geometry>
       </collision>
@@ -92,5 +92,5 @@
         <origin xyz="0 0 0" rpy="0 0 0"/>
         <geometry>
-          <mesh filename="${selector['left_container_jaw']['mesh']}"/>
+          <mesh filename="file://$(find manipulator_description)/meshes/manipulator/left_container_jaw.STL"/>
         </geometry>
         <material name="left_container_jaw_color">
@@ -102,5 +102,5 @@
         <origin xyz="0 0 0" rpy="0 0 0"/>
         <geometry>
-          <mesh filename="${selector['left_container_jaw']['mesh']}"/>
+          <mesh filename="file://$(find manipulator_description)/meshes/manipulator/left_container_jaw.STL"/>
         </geometry>
       </collision>
@@ -157,5 +157,5 @@
         <origin xyz="0 0 0" rpy="0 0 0"/>
         <geometry>
-          <mesh filename="${selector['right_container_jaw']['mesh']}"/>
+          <mesh filename="file://$(find manipulator_description)/meshes/manipulator/right_container_jaw.STL"/>
         </geometry>
         <material name="right_container_jaw_color">
@@ -167,5 +167,5 @@
         <origin xyz="0 0 0" rpy="0 0 0"/>
         <geometry>
-          <mesh filename="${selector['right_container_jaw']['mesh']}"/>
+          <mesh filename="file://$(find manipulator_description)/meshes/manipulator/right_container_jaw.STL"/>
         </geometry>
       </collision>
@@ -227,5 +227,5 @@
         <origin xyz="0 0 0" rpy="0 0 0"/>
         <geometry>
-          <mesh filename="${selector['gripper']['mesh']}"/>
+          <mesh filename="file://$(find manipulator_description)/meshes/manipulator/gripper.STL"/>
         </geometry>
         <material name="gripper_color">
@@ -237,5 +237,5 @@
         <origin xyz="0 0 0" rpy="0 0 0"/>
         <geometry>
-          <mesh filename="${selector['gripper']['mesh']}"/>
+          <mesh filename="file://$(find manipulator_description)/meshes/manipulator/gripper.STL"/>
         </geometry>
       </collision>

File: ros2_ws/src/manipulator_description/urdf/robot.urdf.xacro (robot description, xacro)
@@ -20,5 +20,6 @@
   <!-- Instantiate manipulator (creates base_link and entire manipulator tree) -->
   <xacro:manipulator
-    config_file="$(find manipulator_description)/config/manipulator_params.yaml"/>
+    config_file="$(find manipulator_description)/config/manipulator_params.yaml"
+    sim="true"/>
   <!-- Fixed joint: world -> base_link -->
   <joint name="world_to_base" type="fixed">

Commit message: epics and architecture improved and corrected

File: ros2_ws/src/manipulator_description/urdf/manipulator/manipulator.urdf.xacro (robot description, xacro)
@@ -47,6 +47,8 @@
       config_file="${config_file}"/>
     <!-- 4. ROS2 CONTROL: Hardware interfaces and controllers -->
+    <!-- Uses soft limits (safety_controller) from config_file for command interface limits -->
     <xacro:manipulator_ros2_control
       name="manipulator_system"
+      config_file="${config_file}"
       sim="${sim}"/>
   </xacro:macro>

File: ros2_ws/src/manipulator_description/urdf/manipulator/ros2_control.xacro (robot description, xacro)
@@ -4,9 +4,16 @@
     ROS2 Control Hardware Interface Configuration
     Defines hardware interfaces for the manipulator joints:
-    - Command interfaces: position, velocity
+    - Command interfaces: position, velocity (using SOFT LIMITS from safety_controller)
     - State interfaces: position, velocity
     Uses gazebo_ros2_control for simulation
+    IMPORTANT: Command interface limits use safety_controller soft limits from manipulator_params.yaml
+    This ensures controllers respect operational safety margins, not just physical limits.
   -->
-  <xacro:macro name="manipulator_ros2_control" params="name sim:=true">
+  <xacro:macro name="manipulator_ros2_control" params="name config_file sim:=true">
+    <!-- Load parameters from YAML (same source as URDF joints) -->
+    <xacro:property name="params" value="${xacro.load_yaml(config_file)}"/>
+    <xacro:property name="base" value="${params['base_assembly']}"/>
+    <xacro:property name="selector" value="${params['selector_assembly']}"/>
+    <xacro:property name="picker" value="${params['picker_assembly']}"/>
     <ros2_control name="${name}" type="system">
       <!-- Hardware plugin selection based on sim parameter -->
@@ -29,13 +36,46 @@
       <!-- BASE ASSEMBLY JOINT -->
       <!-- ============================================================ -->
-      <!-- base_main_frame_joint (X-axis railway) -->
+      <!-- base_main_frame_joint (X-axis railway) - uses soft limits -->
       <joint name="base_main_frame_joint">
         <command_interface name="position">
-          <param name="min">0.0</param>
-          <param name="max">4.0</param>
+          <param name="min">${base['base_main_frame_joint']['safety_controller']['soft_lower']}</param>
+          <param name="max">${base['base_main_frame_joint']['safety_controller']['soft_upper']}</param>
         </command_interface>
         <command_interface name="velocity">
-          <param name="min">-2.0</param>
-          <param name="max">2.0</param>
+          <param name="min">-${base['base_main_frame_joint']['limits']['velocity']}</param>
+          <param name="max">${base['base_main_frame_joint']['limits']['velocity']}</param>
+        </command_interface>
+        <state_interface name="position">
+          <param name="initial_value">${base['base_main_frame_joint']['safety_controller']['soft_lower']}</param>
+        </state_interface>
+        <state_interface name="velocity"/>
+      </joint>
+      <!-- ============================================================ -->
+      <!-- SELECTOR ASSEMBLY JOINTS -->
+      <!-- ============================================================ -->
+      <!-- main_frame_selector_frame_joint (Z-axis vertical) - uses soft limits -->
+      <joint name="main_frame_selector_frame_joint">
+        <command_interface name="position">
+          <param name="min">${selector['main_frame_selector_frame_joint']['safety_controller']['soft_lower']}</param>
+          <param name="max">${selector['main_frame_selector_frame_joint']['safety_controller']['soft_upper']}</param>
+        </command_interface>
+        <command_interface name="velocity">
+          <param name="min">-${selector['main_frame_selector_frame_joint']['limits']['velocity']}</param>
+          <param name="max">${selector['main_frame_selector_frame_joint']['limits']['velocity']}</param>
+        </command_interface>
+        <state_interface name="position">
+          <param name="initial_value">${selector['main_frame_selector_frame_joint']['safety_controller']['soft_lower']}</param>
+        </state_interface>
+        <state_interface name="velocity"/>
+      </joint>
+      <!-- selector_left_container_jaw_joint (left container jaw) - uses soft limits -->
+      <joint name="selector_left_container_jaw_joint">
+        <command_interface name="position">
+          <param name="min">${selector['selector_left_container_jaw_joint']['safety_controller']['soft_lower']}</param>
+          <param name="max">${selector['selector_left_container_jaw_joint']['safety_controller']['soft_upper']}</param>
+        </command_interface>
+        <command_interface name="velocity">
+          <param name="min">-${selector['selector_left_container_jaw_joint']['limits']['velocity']}</param>
+          <param name="max">${selector['selector_left_container_jaw_joint']['limits']['velocity']}</param>
         </command_interface>
         <state_interface name="position">
@@ -44,31 +84,14 @@
         <state_interface name="velocity"/>
       </joint>
-      <!-- ============================================================ -->
-      <!-- SELECTOR ASSEMBLY JOINTS -->
-      <!-- ============================================================ -->
-      <!-- main_frame_selector_frame_joint (Z-axis vertical) -->
-      <joint name="main_frame_selector_frame_joint">
+      <!-- selector_right_container_jaw_joint (right container jaw) - uses soft limits -->
+      <!-- Note: Was mimic joint, but dartsim doesn't support mimic, so controlled independently -->
+      <joint name="selector_right_container_jaw_joint">
         <command_interface name="position">
-          <param name="min">-0.01</param>
-          <param name="max">1.5</param>
+          <param name="min">${selector['selector_right_container_jaw_joint']['safety_controller']['soft_lower']}</param>
+          <param name="max">${selector['selector_right_container_jaw_joint']['safety_controller']['soft_upper']}</param>
         </command_interface>
         <command_interface name="velocity">
-          <param name="min">-2.0</param>
-          <param name="max">2.0</param>
-        </command_interface>
-        <state_interface name="position">
-          <param name="initial_value">0.05</param>
-        </state_interface>
-        <state_interface name="velocity"/>
-      </joint>
-      <!-- selector_left_container_jaw_joint (left container jaw) -->
-      <joint name="selector_left_container_jaw_joint">
-        <command_interface name="position">
-          <param name="min">-0.2</param>
-          <param name="max">0.2</param>
-        </command_interface>
-        <command_interface name="velocity">
-          <param name="min">-1.0</param>
-          <param name="max">1.0</param>
+          <param name="min">-${selector['selector_right_container_jaw_joint']['limits']['velocity']}</param>
+          <param name="max">${selector['selector_right_container_jaw_joint']['limits']['velocity']}</param>
         </command_interface>
         <state_interface name="position">
@@ -77,29 +100,13 @@
         <state_interface name="velocity"/>
       </joint>
-      <!-- selector_right_container_jaw_joint (right container jaw) -->
-      <!-- Note: Was mimic joint, but dartsim doesn't support mimic, so controlled independently -->
-      <joint name="selector_right_container_jaw_joint">
+      <!-- selector_frame_gripper_joint (Y-axis magnet holder) - uses soft limits -->
+      <joint name="selector_frame_gripper_joint">
         <command_interface name="position">
-          <param name="min">-0.2</param>
-          <param name="max">0.2</param>
+          <param name="min">${selector['selector_frame_gripper_joint']['safety_controller']['soft_lower']}</param>
+          <param name="max">${selector['selector_frame_gripper_joint']['safety_controller']['soft_upper']}</param>
         </command_interface>
         <command_interface name="velocity">
-          <param name="min">-1.0</param>
-          <param name="max">1.0</param>
-        </command_interface>
-        <state_interface name="position">
-          <param name="initial_value">0.0</param>
-        </state_interface>
-        <state_interface name="velocity"/>
-      </joint>
-      <!-- selector_frame_gripper_joint (Y-axis magnet holder) -->
-      <joint name="selector_frame_gripper_joint">
-        <command_interface name="position">
-          <param name="min">-0.4</param>
-          <param name="max">0.4</param>
-        </command_interface>
-        <command_interface name="velocity">
-          <param name="min">-1.0</param>
-          <param name="max">1.0</param>
+          <param name="min">-${selector['selector_frame_gripper_joint']['limits']['velocity']}</param>
+          <param name="max">${selector['selector_frame_gripper_joint']['limits']['velocity']}</param>
         </command_interface>
         <state_interface name="position">
@@ -111,28 +118,28 @@
       <!-- PICKER ASSEMBLY JOINTS -->
       <!-- ============================================================ -->
-      <!-- selector_frame_picker_frame_joint (Z-axis picker vertical) -->
+      <!-- selector_frame_picker_frame_joint (Z-axis picker vertical) - uses soft limits -->
       <joint name="selector_frame_picker_frame_joint">
         <command_interface name="position">
-          <param name="min">-0.01</param>
-          <param name="max">0.3</param>
+          <param name="min">${picker['selector_frame_picker_frame_joint']['safety_controller']['soft_lower']}</param>
+          <param name="max">${picker['selector_frame_picker_frame_joint']['safety_controller']['soft_upper']}</param>
         </command_interface>
         <command_interface name="velocity">
-          <param name="min">-1.0</param>
-          <param name="max">1.0</param>
+          <param name="min">-${picker['selector_frame_picker_frame_joint']['limits']['velocity']}</param>
+          <param name="max">${picker['selector_frame_picker_frame_joint']['limits']['velocity']}</param>
         </command_interface>
         <state_interface name="position">
-          <param name="initial_value">0.05</param>
+          <param name="initial_value">${picker['selector_frame_picker_frame_joint']['safety_controller']['soft_lower']}</param>
         </state_interface>
         <state_interface name="velocity"/>
       </joint>
-      <!-- picker_frame_picker_rail_joint (Y-axis picker rail) -->
+      <!-- picker_frame_picker_rail_joint (Y-axis picker rail) - uses soft limits -->
       <joint name="picker_frame_picker_rail_joint">
         <command_interface name="position">
-          <param name="min">-0.3</param>
-          <param name="max">0.3</param>
+          <param name="min">${picker['picker_frame_picker_rail_joint']['safety_controller']['soft_lower']}</param>
+          <param name="max">${picker['picker_frame_picker_rail_joint']['safety_controller']['soft_upper']}</param>
         </command_interface>
         <command_interface name="velocity">
-          <param name="min">-1.0</param>
-          <param name="max">1.0</param>
+          <param name="min">-${picker['picker_frame_picker_rail_joint']['limits']['velocity']}</param>
+          <param name="max">${picker['picker_frame_picker_rail_joint']['limits']['velocity']}</param>
         </command_interface>
         <state_interface name="position">
@@ -141,31 +148,31 @@
         <state_interface name="velocity"/>
       </joint>
-      <!-- picker_rail_picker_base_joint (X-axis picker slider) -->
+      <!-- picker_rail_picker_base_joint (X-axis picker slider) - uses soft limits -->
       <joint name="picker_rail_picker_base_joint">
         <command_interface name="position">
-          <param name="min">0.0</param>
-          <param name="max">0.25</param>
+          <param name="min">${picker['picker_rail_picker_base_joint']['safety_controller']['soft_lower']}</param>
+          <param name="max">${picker['picker_rail_picker_base_joint']['safety_controller']['soft_upper']}</param>
         </command_interface>
         <command_interface name="velocity">
-          <param name="min">-1.0</param>
-          <param name="max">1.0</param>
+          <param name="min">-${picker['picker_rail_picker_base_joint']['limits']['velocity']}</param>
+          <param name="max">${picker['picker_rail_picker_base_joint']['limits']['velocity']}</param>
         </command_interface>
         <state_interface name="position">
-          <param name="initial_value">0.0</param>
+          <param name="initial_value">${picker['picker_rail_picker_base_joint']['safety_controller']['soft_lower']}</param>
         </state_interface>
         <state_interface name="velocity"/>
       </joint>
-      <!-- picker_base_picker_jaw_joint (X-axis picker extension) -->
+      <!-- picker_base_picker_jaw_joint (X-axis picker extension) - uses soft limits -->
       <joint name="picker_base_picker_jaw_joint">
         <command_interface name="position">
-          <param name="min">0.0</param>
-          <param name="max">0.2</param>
+          <param name="min">${picker['picker_base_picker_jaw_joint']['safety_controller']['soft_lower']}</param>
+          <param name="max">${picker['picker_base_picker_jaw_joint']['safety_controller']['soft_upper']}</param>
         </command_interface>
         <command_interface name="velocity">
-          <param name="min">-1.0</param>
-          <param name="max">1.0</param>
+          <param name="min">-${picker['picker_base_picker_jaw_joint']['limits']['velocity']}</param>
+          <param name="max">${picker['picker_base_picker_jaw_joint']['limits']['velocity']}</param>
         </command_interface>
         <state_interface name="position">
-          <param name="initial_value">0.0</param>
+          <param name="initial_value">${picker['picker_base_picker_jaw_joint']['safety_controller']['soft_lower']}</param>
         </state_interface>
         <state_interface name="velocity"/>
